Commit message: 9.4

File: phc/data/assets/robot/ehr03/urdf/ehr03_lp.urdf (robot description, URDF)
Before this commit: robot ehr_03, 32 links, 31 joints
Links:
- added link neck_l1, mass 0.292159909832987; collision mesh filename=../meshes/neck_l1_fixed.STL; visual mesh filename=../meshes/neck_l1_fixed.STL
- added link neck_l2, mass 2.13608587519163; collision mesh filename=../meshes/neck_l2_fixed.STL; visual mesh filename=../meshes/neck_l2_fixed.STL
Joints:
- added joint neck_1: type revolute, parent torso_l3, child neck_l1, origin xyz=0.0335 0 0.409 rpy=0 0 0, axis 0 0 1, limit lower=-1.57 upper=1.57 effort=0 velocity=0
- added joint neck_2: type revolute, parent neck_l1, child neck_l2, origin xyz=0 0 0.047 rpy=0 0 0, axis 0 1 0, limit lower=-0.523 upper=0.523 effort=0 velocity=0
